File: nodular-base/base-can.kicad_sch (KiCad schematic)
At the start: 1 part, among them U5 MAX3051

Commit message: WIP layout for base
Parts:
- added C3: 100nF, Capacitor_SMD:C_0402_1005Metric, symbol Device:C
- added R12: R, Resistor_SMD:R_0402_1005Metric, symbol Device:R
- added R13: R, Resistor_SMD:R_0603_1608Metric, symbol Device:R
Connections:
- net GND: now reaches U5.2 (GND)
- net GND: now also C3.2, R12.2
- net at U5.3 (VDD): now also C3.1
- net at U5.7 (CANH): now also R13.1
- net at U5.8 (RS): now also R12.1
Changed lines of the file:
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@@
 (kicad_sch (version 20230121) (generator eeschema)
   (paper "A4")
+  (junction (at 106.68 95.25) (diameter 0) (color 0 0 0 0)
+  )
+  (wire (pts (xy 106.68 62.23) (xy 106.68 72.39))
+    (stroke (width 0) (type default))
+  )
+  (wire (pts (xy 97.79 62.23) (xy 106.68 62.23))
+    (stroke (width 0) (type default))
+  )
+  (wire (pts (xy 93.98 95.25) (xy 106.68 95.25))
+    (stroke (width 0) (type default))
+  )
+  (wire (pts (xy 106.68 95.25) (xy 106.68 92.71))
+    (stroke (width 0) (type default))
+  )
+  (wire (pts (xy 119.38 80.01) (xy 129.54 80.01))
+    (stroke (width 0) (type default))
+  )
+  (symbol (lib_id "power:GND") (at 106.68 95.25 0) (unit 1)
+    (in_bom yes) (on_board yes) (dnp no) (fields_autoplaced)
+    (property "Reference" "#PWR028" (at 106.68 101.6 0)
+      (effects (font (size 1.27 1.27)) hide)
+    )
+    (property "Value" "GND" (at 106.68 100.33 0)
+      (effects (font (size 1.27 1.27)))
+    )
+    (property "Footprint" "" (at 106.68 95.25 0)
+      (effects (font (size 1.27 1.27)) hide)
+    )
+    (property "Datasheet" "" (at 106.68 95.25 0)
+      (effects (font (size 1.27 1.27)) hide)
+    )
+    (pin "1")
+    (instances
+      (project "nodular-base"
+        (path "/6dcb0502-87e2-4c28-9ce8-81aab8925f06/e3861226-82ef-4af3-8bf9-5142ff955f1b"
+          (reference "#PWR028") (unit 1)
+        )
+      )
+    )
+  )
+  (symbol (lib_id "power:GND") (at 97.79 69.85 0) (unit 1)
+    (in_bom yes) (on_board yes) (dnp no)
+    (property "Reference" "#PWR029" (at 97.79 76.2 0)
+      (effects (font (size 1.27 1.27)) hide)
+    )
+    (property "Value" "GND" (at 101.6 71.12 0)
+      (effects (font (size 1.27 1.27)))
+    )
+    (property "Footprint" "" (at 97.79 69.85 0)
+      (effects (font (size 1.27 1.27)) hide)
+    )
+    (property "Datasheet" "" (at 97.79 69.85 0)
+      (effects (font (size 1.27 1.27)) hide)
+    )
+    (pin "1")
+    (instances
+      (project "nodular-base"
+        (path "/6dcb0502-87e2-4c28-9ce8-81aab8925f06/e3861226-82ef-4af3-8bf9-5142ff955f1b"
+          (reference "#PWR029") (unit 1)
+        )
+      )
+    )
+  )
+  (symbol (lib_id "Device:C") (at 97.79 66.04 0) (unit 1)
+    (in_bom yes) (on_board yes) (dnp no)
+    (property "Reference" "C3" (at 97.79 63.5 0)
+      (effects (font (size 1.27 1.27)) (justify left))
+    )
+    (property "Value" "100nF" (at 97.79 68.58 0)
+      (effects (font (size 1.27 1.27)) (justify left))
+    )
+    (property "Footprint" "Capacitor_SMD:C_0402_1005Metric" (at 98.7552 69.85 0)
+      (effects (font (size 1.27 1.27)) hide)
+    )
+    (property "Datasheet" "~" (at 97.79 66.04 0)
+      (effects (font (size 1.27 1.27)) hide)
+    )
+    (pin "1")
+    (pin "2")
+    (instances
+      (project "nodular-base"
+        (path "/6dcb0502-87e2-4c28-9ce8-81aab8925f06"
+          (reference "C3") (unit 1)
+        )
+        (path "/6dcb0502-87e2-4c28-9ce8-81aab8925f06/e3861226-82ef-4af3-8bf9-5142ff955f1b"
+          (reference "C16") (unit 1)
+        )
+      )
+    )
+  )
   (symbol (lib_id "Interface_UART:MAX3051") (at 106.68 82.55 0) (unit 1)
     (in_bom yes) (on_board yes) (dnp no) (fields_autoplaced)
@@
         )
       )
+    )
+  )
+  (symbol (lib_id "Device:R") (at 129.54 83.82 0) (unit 1)
+    (in_bom yes) (on_board yes) (dnp no) (fields_autoplaced)
+    (property "Reference" "R13" (at 132.08 82.55 0)
+      (effects (font (size 1.27 1.27)) (justify left))
+    )
+    (property "Value" "R" (at 132.08 85.09 0)
+      (effects (font (size 1.27 1.27)) (justify left))
+    )
+    (property "Footprint" "Resistor_SMD:R_0603_1608Metric" (at 127.762 83.82 90)
+      (effects (font (size 1.27 1.27)) hide)
+    )
+    (property "Datasheet" "~" (at 129.54 83.82 0)
+      (effects (font (size 1.27 1.27)) hide)
+    )
+    (pin "1")
+    (pin "2")
+    (instances
+      (project "nodular-base"
+        (path "/6dcb0502-87e2-4c28-9ce8-81aab8925f06/e3861226-82ef-4af3-8bf9-5142ff955f1b"
+          (reference "R13") (unit 1)
+        )
+      )
+    )
+  )
+  (symbol (lib_id "Device:R") (at 93.98 91.44 0) (unit 1)
+    (in_bom yes) (on_board yes) (dnp no)
+    (property "Reference" "R12" (at 91.44 90.17 0)
+      (effects (font (size 1.27 1.27)) (justify right))
+    )
+    (property "Value" "R" (at 91.44 92.71 0)
+      (effects (font (size 1.27 1.27)) (justify right))
+    )
+    (property "Footprint" "Resistor_SMD:R_0402_1005Metric" (at 92.202 91.44 90)
+      (effects (font (size 1.27 1.27)) hide)
+    )
+    (property "Datasheet" "~" (at 93.98 91.44 0)
+      (effects (font (size 1.27 1.27)) hide)
+    )
+    (pin "1")
+    (pin "2")
+    (instances
+      (project "nodular-base"
+        (path "/6dcb0502-87e2-4c28-9ce8-81aab8925f06/e3861226-82ef-4af3-8bf9-5142ff955f1b"
+          (reference "R12") (unit 1)
+        )
+      )
