File: tildagon-base/tildagon-base.kicad_sch (KiCad schematic)
At the start: 31 parts, among them J11 Conn_01x08_Pin, SW1 SW_Push, SW2 SW_Push, SW3 SW_Push, U1 ESP32-S3-PICO-1-N8R2

Commit message: Final production design for emf2024
Parts:
- removed N1: Housing, tildagon:bartholomew, symbol Mechanical:Housing
