File: tildagon-base/tildagon-base.kicad_pcb (KiCad board)
At the start: 4 copper layers, 83.1 x 92.5 mm, 183 parts, among them J1 Conn_02x10_Counter_Clockwise, J10 Conn_01x02_MountingPin, J11 Conn_01x08_Pin, J2 Conn_02x10_Counter_Clockwise, J3 Conn_02x10_Counter_Clockwise, J4 Conn_02x10_Counter_Clockwise, J5 Conn_02x10_Counter_Clockwise, J6 Conn_02x10_Counter_Clockwise, J7 USB_C_Receptacle_USB2.0, J8 USB_C_Receptacle_USB2.0, J9 Conn_01x30_MountingPin, SW1 SW_Push, SW2 SW_Push, SW3 SW_Push, U1 ESP32-S3-PICO-1-N8R2, U10 MT9700, U11 MT9700, U12 MT9700, U13 MT9700, U14 MT9700, U15 74LVC1G04, U16 RCLAMP0524P-ES, U17 RCLAMP0524P-ES, U18 RCLAMP0524P-ES, U19 74LVC1G04, U2 FUSB302BMPX, U20 RCLAMP0524P-ES, U21 RCLAMP0524P-ES, U22 RCLAMP0524P-ES, U23 74LVC1G04, U24 AW9523B, U25 AW9523B, U26 AW9523B, U27 RCLAMP0524P-ES, U28 RCLAMP0524P-ES, U29 RCLAMP0524P-ES, U3 BQ25895RTW, U30 RCLAMP0524P-ES, U31 74LVC1G04, U32 74LVC1G04, U33 74LVC1G04, U34 RCLAMP0524P-ES, U35 RCLAMP0524P-ES, U36 RCLAMP0524P-ES, U37 RCLAMP0524P-ES, U38 RCLAMP0524P-ES, U39 RCLAMP0524P-ES, U4 TCA9548APWR, U40 RCLAMP0524P-ES, U41 RCLAMP0524P-ES, U42 RCLAMP0524P-ES, U43 TLV62595DMQR, U44 RCLAMP0524P-ES, U45 RCLAMP0524P-ES, U46 RCLAMP0524P-ES, U47 RCLAMP0524P-ES, U48 RCLAMP0524P-ES, U49 RCLAMP0524P-ES, U5 FUSB302BMPX, U50 TS3USB221A, U51 MT9700, U52 LSM6DS3, U6 74LVC1G17, U7 SC7A20, U8 MT9700, U9 MT9700

Commit message: Update base schematic files to 2026 version, regenerate PDF Update hexpansion project file version to fix trace visibility
Parts:
- U52: value LSM6DS3 -> BMI270
