File: tildagon-base/base-i2c.kicad_sch (KiCad schematic)
At the start: 6 parts, among them U4 TCA9548APWR, U52 LSM6DS3, U7 SC7A20

Commit message: Update base schematic files to 2026 version, regenerate PDF Update hexpansion project file version to fix trace visibility
Parts:
- U52: value LSM6DS3 -> BMI270
Changed lines of the file:
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@@
 (kicad_sch
-	(version 20231120)
+	(version 20250114)
 	(generator "eeschema")
-	(generator_version "8.0")
+	(generator_version "9.0")
 	(paper "A4")
 	(junction
@@
 	(label "3V3_SYS"
 		(at 113.03 52.07 0)
-		(fields_autoplaced yes)
 		(effects
 			(font
@@
 	(label "3V3_SYS"
 		(at 234.95 95.25 180)
-		(fields_autoplaced yes)
 		(effects
 			(font
@@
 	(label "SCL_SYS"
 		(at 234.95 92.71 180)
-		(fields_autoplaced yes)
 		(effects
 			(font
@@
 	(label "SCL_SYS"
 		(at 176.53 74.93 180)
-		(fields_autoplaced yes)
 		(effects
 			(font
@@
 	(label "3V3_SYS"
 		(at 250.19 72.39 180)
-		(fields_autoplaced yes)
 		(effects
 			(font
@@
 	(label "SDA_SYS"
 		(at 234.95 90.17 180)
-		(fields_autoplaced yes)
 		(effects
 			(font
@@
 	(label "3V3_SYS"
 		(at 102.87 80.01 180)
-		(fields_autoplaced yes)
 		(effects
 			(font
@@
 	(label "3V3_SYS"
 		(at 201.93 59.69 0)
-		(fields_autoplaced yes)
 		(effects
 			(font
@@
 	(label "3V3_SYS"
 		(at 210.82 77.47 0)
-		(fields_autoplaced yes)
 		(effects
 			(font
@@
 	(label "SDA_SYS"
 		(at 176.53 69.85 180)
-		(fields_autoplaced yes)
 		(effects
 			(font
@@
 	(label "3V3_SYS"
 		(at 146.05 34.29 0)
-		(fields_autoplaced yes)
 		(effects
 			(font
@@
 		(shape input)
 		(at 142.24 34.29 180)
-		(fields_autoplaced yes)
 		(effects
 			(font
@@
 		(shape output)
 		(at 123.19 82.55 0)
-		(fields_autoplaced yes)
 		(effects
 			(font
@@
 		(shape bidirectional)
 		(at 123.19 80.01 0)
-		(fields_autoplaced yes)
 		(effects
 			(font
@@
 		(shape bidirectional)
 		(at 102.87 59.69 180)
-		(fields_autoplaced yes)
 		(effects
 			(font
@@
 		(shape output)
 		(at 123.19 92.71 0)
-		(fields_autoplaced yes)
 		(effects
 			(font
@@
 		(shape output)
 		(at 123.19 87.63 0)
-		(fields_autoplaced yes)
 		(effects
 			(font
@@
 		(shape bidirectional)
 		(at 123.19 69.85 0)
-		(fields_autoplaced yes)
 		(effects
 			(font
@@
 		(shape input)
 		(at 102.87 69.85 180)
-		(fields_autoplaced yes)
 		(effects
 			(font
@@
 		(shape bidirectional)
 		(at 208.28 69.85 0)
-		(fields_autoplaced yes)
 		(effects
 			(font
@@
 		(shape output)
 		(at 123.19 67.31 0)
-		(fields_autoplaced yes)
 		(effects
 			(font
@@
 		(shape bidirectional)
 		(at 123.19 74.93 0)
-		(fields_autoplaced yes)
 		(effects
 			(font
@@
 		(shape input)
 		(at 102.87 57.15 180)
-		(fields_autoplaced yes)
 		(effects
 			(font
@@
 		(shape output)
 		(at 123.19 57.15 0)
-		(fields_autoplaced yes)
 		(effects
 			(font
@@
 		(shape bidirectional)
 		(at 123.19 90.17 0)
-		(fields_autoplaced yes)
 		(effects
 			(font
@@
 		(shape output)
 		(at 123.19 72.39 0)
-		(fields_autoplaced yes)
 		(effects
 			(font
@@
 		(shape bidirectional)
 		(at 123.19 64.77 0)
-		(fields_autoplaced yes)
 		(effects
 			(font
@@
 		(shape bidirectional)
 		(at 123.19 95.25 0)
-		(fields_autoplaced yes)
 		(effects
 			(font
@@
 		(shape output)
 		(at 123.19 77.47 0)
-		(fields_autoplaced yes)
 		(effects
 			(font
@@
 		(shape bidirectional)
 		(at 123.19 85.09 0)
-		(fields_autoplaced yes)
 		(effects
 			(font
@@
 		(shape bidirectional)
 		(at 123.19 59.69 0)
-		(fields_autoplaced yes)
 		(effects
 			(font
@@
 		(shape bidirectional)
 		(at 265.43 80.01 0)
-		(fields_autoplaced yes)
 		(effects
 			(font
@@
 		(shape output)
 		(at 123.19 62.23 0)
-		(fields_autoplaced yes)
 		(effects
 			(font
@@
 			)
 		)
-		(property "Value" "LSM6DS3"
+		(property "Value" "BMI270"
 			(at 252.3841 105.41 0)
 			(effects
@@
 			)
 		)
-		(property "Datasheet" "https://www.st.com/resource/en/datasheet/lsm6ds3tr-c.pdf"
+		(property "Datasheet" "https://www.bosch-sensortec.com/media/boschsensortec/downloads/datasheets/bst-bmi270-ds000.pdf"
 			(at 252.73 104.14 0)
 			(effects
