File: tildagon-base/bot-top-link.kicad_sch (KiCad schematic)
At the start: 18 parts, among them J9 Conn_01x30_MountingPin, U14 MT9700, U44 RCLAMP0524P-ES, U45 RCLAMP0524P-ES, U46 RCLAMP0524P-ES, U47 RCLAMP0524P-ES, U48 RCLAMP0524P-ES, U6 74LVC1G17

Commit message: Update base schematic files to 2026 version, regenerate PDF Update hexpansion project file version to fix trace visibility
Parts:
- renumbered D14 to D2
Changed lines of the file:
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@@
 (kicad_sch
-	(version 20231120)
+	(version 20250114)
 	(generator "eeschema")
-	(generator_version "8.0")
+	(generator_version "9.0")
 	(paper "A4")
 	(junction
@@
 	(label "GND"
 		(at 41.91 120.65 0)
-		(fields_autoplaced yes)
 		(effects
 			(font
@@
 	(label "TOP_VBAT_SW"
 		(at 157.48 41.91 0)
-		(fields_autoplaced yes)
 		(effects
 			(font
@@
 	(label "GND"
 		(at 41.91 57.15 0)
-		(fields_autoplaced yes)
 		(effects
 			(font
@@
 	(label "TOP_VBAT_SW"
 		(at 41.91 52.07 0)
-		(fields_autoplaced yes)
 		(effects
 			(font
@@
 	(label "TOP_VBAT_SW"
 		(at 41.91 54.61 0)
-		(fields_autoplaced yes)
 		(effects
 			(font
@@
 	(label "TOP_VBAT_SW"
 		(at 115.57 39.37 0)
-		(fields_autoplaced yes)
 		(effects
 			(font
@@
 	(label "GND"
 		(at 41.91 81.28 0)
-		(fields_autoplaced yes)
 		(effects
 			(font
@@
 	(label "TOP_VBAT_SW"
 		(at 138.43 72.39 0)
-		(fields_autoplaced yes)
 		(effects
 			(font
@@
 	(label "LED_DATA_TOP"
 		(at 41.91 49.53 0)
-		(fields_autoplaced yes)
 		(effects
 			(font
@@
 	(label "GND"
 		(at 41.91 118.11 0)
-		(fields_autoplaced yes)
 		(effects
 			(font
@@
 	(label "LED_DATA_TOP"
 		(at 172.72 49.53 0)
-		(fields_autoplaced yes)
 		(effects
 			(font
@@
 	(label "GND"
 		(at 41.91 95.25 0)
-		(fields_autoplaced yes)
 		(effects
 			(font
@@
 	(label "GND"
 		(at 41.91 46.99 0)
-		(fields_autoplaced yes)
 		(effects
 			(font
@@
 		(shape bidirectional)
 		(at 44.45 114.3 0)
-		(fields_autoplaced yes)
 		(effects
 			(font
@@
 		(shape bidirectional)
 		(at 48.26 91.44 0)
-		(fields_autoplaced yes)
 		(effects
 			(font
@@
 		(shape bidirectional)
 		(at 48.26 104.14 0)
-		(fields_autoplaced yes)
 		(effects
 			(font
@@
 		(shape bidirectional)
 		(at 48.26 99.06 0)
-		(fields_autoplaced yes)
 		(effects
 			(font
@@
 		(shape input)
 		(at 105.41 49.53 180)
-		(fields_autoplaced yes)
 		(effects
 			(font
@@
 		(shape bidirectional)
 		(at 48.26 101.6 0)
-		(fields_autoplaced yes)
 		(effects
 			(font
@@
 		(shape bidirectional)
 		(at 44.45 111.76 0)
-		(fields_autoplaced yes)
 		(effects
 			(font
@@
 		(shape bidirectional)
 		(at 41.91 64.77 0)
-		(fields_autoplaced yes)
 		(effects
 			(font
@@
 		(shape bidirectional)
 		(at 48.26 96.52 0)
-		(fields_autoplaced yes)
 		(effects
 			(font
@@
 		(shape bidirectional)
 		(at 41.91 72.39 0)
-		(fields_autoplaced yes)
 		(effects
 			(font
@@
 		(shape input)
 		(at 101.6 69.85 180)
-		(fields_autoplaced yes)
 		(effects
 			(font
@@
 		(shape bidirectional)
 		(at 48.26 86.36 0)
-		(fields_autoplaced yes)
 		(effects
 			(font
@@
 		(shape bidirectional)
 		(at 41.91 69.85 0)
-		(fields_autoplaced yes)
 		(effects
 			(font
@@
 		(shape bidirectional)
 		(at 44.45 109.22 0)
-		(fields_autoplaced yes)
 		(effects
 			(font
@@
 		(shape bidirectional)
 		(at 41.91 67.31 0)
-		(fields_autoplaced yes)
 		(effects
 			(font
@@
 		(shape bidirectional)
 		(at 48.26 88.9 0)
-		(fields_autoplaced yes)
 		(effects
 			(font
@@
 		(shape bidirectional)
 		(at 41.91 62.23 0)
-		(fields_autoplaced yes)
 		(effects
 			(font
@@
 		(shape bidirectional)
 		(at 48.26 83.82 0)
-		(fields_autoplaced yes)
 		(effects
 			(font
@@
 		(shape bidirectional)
 		(at 41.91 59.69 0)
-		(fields_autoplaced yes)
 		(effects
 			(font
@@
 		(shape input)
 		(at 106.68 85.09 180)
-		(fields_autoplaced yes)
 		(effects
 			(font
@@
 		(shape bidirectional)
 		(at 44.45 106.68 0)
-		(fields_autoplaced yes)
 		(effects
 			(font
@@
 		(shape bidirectional)
 		(at 43.18 76.2 0)
-		(fields_autoplaced yes)
 		(effects
 			(font
@@
 		(on_board yes)
 		(dnp no)
-		(property "Reference" "D14"
+		(property "Reference" "D2"
 			(at 161.29 43.18 0)
 			(effects
